Commit message: with npcs semi working

File: urdf/truck.urdf (robot description, URDF)
Before this commit: robot truck, 2 links, 1 joints
Links:
- added link base_link, mass 1
Joints:
- added joint base_link_joint: type fixed, parent base_link, child tractor, origin xyz=1.45 0 0 rpy=0 0 1.57, axis 1 0 0
