Commit message: truck with lidar!!!

File: urdf/ego_vehicle.xacro (robot description, xacro)
@@ -1,3 +1,129 @@
 <?xml version="1.0"?>
 <robot xmlns:xacro="http://www.ros.org/wiki/xacro" name="ego_vehicle">
+    <xacro:include filename="$(find my_truckie)/urdf/lidar.plugins.xacro" />
+    <xacro:property name="scale_factor" value="6.0" />
+    <xacro:property name="laser_size_x" value="0.03"/>
+    <xacro:property name="laser_size_y" value="0.03"/>
+    <xacro:property name="laser_size_z" value="0.04"/>
+    <xacro:property name="laser_origin_x" value="0.065"/>
+    <xacro:property name="laser_origin_y" value="0"/>
+    <xacro:property name="laser_origin_z" value="0.025"/>
+    <xacro:macro name="default_inertial" params="mass">
+        <inertial>
+        <mass value="${mass}"/>
+        <inertia ixx="1.0" ixy="0.0" ixz="0.0" iyy="1.0" iyz="0.0" izz="1.0"/>
+        </inertial>
+    </xacro:macro>
+    <link name="base_footprint">
+        <inertial>
+            <mass value="0.0001" />
+            <origin xyz="0 0 0" />
+            <inertia ixx="0.0001" ixy="0.0" ixz="0.0"
+                iyy="0.0001" iyz="0.0"
+                izz="0.0001" />
+        </inertial>
+        <visual>
+            <origin xyz="0 0 0" rpy="0 0 0" />
+            <geometry>
+                <box size="0.001 0.001 0.001" />
+            </geometry>
+        </visual>
+    </link>
+    <joint name="base_footprint_joint" type="fixed">
+        <origin xyz="0 0 0" rpy="0 0 0" />
+        <parent link="base_footprint"/>
+        <child link="tractor" />
+    </joint>
+    <!-- Tractor -->
+    <link name="tractor">
+        <visual>
+            <origin xyz="0 0 ${scale_factor*0.25}" rpy="0 0 0"/>
+            <geometry>
+            <box size="${scale_factor*0.5} ${scale_factor*0.5} ${scale_factor*0.5}"/>
+            </geometry>
+            <material name="blue">
+            <color rgba="0 0 1 1"/>
+            </material>
+        </visual>
+        <collision>
+            <origin xyz="0 0 ${scale_factor*0.25}" rpy="0 0 0"/>
+            <geometry>
+            <box size="${scale_factor*0.5} ${scale_factor*0.5} ${scale_factor*0.5}"/>
+            </geometry>
+            <surface>
+            <friction> <!-- friction coefficients must be set to 0 allowing it to move -->
+                <ode>
+                <mu>0</mu>
+                <mu2>0</mu2>
+                </ode>
+            </friction>
+            </surface>
+        </collision>
+        <inertial>
+            <mass value="1"/>
+            <origin xyz="0 0 0" rpy="0 0 0"/>
+            <inertia ixx="1" ixy="0" ixz="0" iyy="1" iyz="0" izz="1"/>
+        </inertial>
+    </link>
+    <!-- Tractor-trailer Joint -->
+    <joint name="hitch_joint" type="revolute">
+        <parent link="tractor"/>
+        <child link="trailer"/>
+        <origin xyz="0 0 0" rpy="0 0 0"/>
+        <axis xyz="0 0 1"/>
+        <limit effort="100" velocity="1.0" lower="-1.5708" upper="1.5708"/>
+    </joint>
+    <!-- Trailer -->
+    <link name="trailer">
+        <visual>
+            <origin xyz="-${scale_factor*0.75} 0 ${scale_factor*0.25}" rpy="0 0 0"/>
+            <geometry>
+            <box size="${scale_factor*1} ${scale_factor*0.5} ${scale_factor*0.5}"/>
+            </geometry>
+            <material name="red">
+            <color rgba="1 0 0 1"/>
+            </material>
+        </visual>
+        <collision>
+            <origin xyz="-${scale_factor*0.75} 0 ${scale_factor*0.25}" rpy="0 0 0"/>
+            <geometry>
+            <box size="${scale_factor*1} ${scale_factor*0.5} ${scale_factor*0.5}"/>
+            </geometry>
+            <surface>
+            <friction> <!-- friction coefficients must be set to 0 allowing it to move -->
+                <ode>
+                <mu>0</mu>
+                <mu2>0</mu2>
+                </ode>
+            </friction>
+            </surface>
+        </collision>
+        <inertial>
+            <mass value="1"/>
+            <origin xyz="0 0 0" rpy="0 0 0"/>
+            <inertia ixx="1" ixy="0" ixz="0" iyy="1" iyz="0" izz="1"/>
+        </inertial>
+    </link>
+    <!--Laser Scan-->
+    <link name="sensor_laser">
+        <visual>
+        <geometry>
+            <mesh filename="package://my_truckie/meshes/hokuyo.dae"/>
+            <!--box size="${laser_size_x} ${laser_size_y} ${laser_size_z}"/-->
+        </geometry>
+        <material name="blue"/>
+        </visual>
+        <collision>
+        <geometry>
+            <box size="${laser_size_x} ${laser_size_y} ${laser_size_z}"/>
+        </geometry>
+        </collision>
+        <xacro:default_inertial mass="0.02"/>
+    </link>
+    <joint name="sensor_laser_joint" type="fixed">
+        <!-- <origin xyz="${laser_origin_x} ${laser_origin_y} ${laser_origin_z}" rpy="0 0 0" /> -->
+        <origin xyz="1.5 0 0.5" rpy="0 0 0" />
+        <parent link="tractor"/>
+        <child link="sensor_laser" />
+    </joint>
 </robot>

Commit message: before applying models dynamics

File: urdf/ego_vehicle.xacro (robot description, xacro)
@@ -127,3 +127,21 @@
         <child link="sensor_laser" />
     </joint>
+    <!-- Joint Controller for Hitch Joint -->
+    <transmission name="trans_hitch_joint">
+        <type>transmission_interface/SimpleTransmission</type>
+        <joint name="hitch_joint">
+        <hardwareInterface>hardware_interface/EffortJointInterface</hardwareInterface>
+        </joint>
+        <actuator name="motor_hitch_joint">
+        <hardwareInterface>hardware_interface/EffortJointInterface</hardwareInterface>
+        <mechanicalReduction>1</mechanicalReduction>
+        </actuator>
+    </transmission>
+    <!-- <plugin name="object_controller" filename="libgazebo_ros_planar_move.so">
+        <commandTopic>cmd_vel</commandTopic>
+        <odometryTopic>odom</odometryTopic>
+        <odometryFrame>odom</odometryFrame>
+        <odometryRate>50.0</odometryRate>
+        <robotBaseFrame>base_footprint</robotBaseFrame>
+    </plugin> -->
 </robot>

File: urdf/lidar.plugins.xacro (robot description, xacro)
@@ -1,35 +1,51 @@
 <?xml version="1.0"?>
 <robot>
-  <!--Gazebo Hokuyo Laser Plugin-->
-  <gazebo reference="sensor_laser">
-    <sensor type="ray" name="head_hokuyo_sensor">
-      <pose>0 0 0 0 0 0</pose>
-      <visualize>true</visualize>
-      <update_rate>40</update_rate>
-      <ray>
-        <scan>
-          <horizontal>
-            <samples>720</samples>
-            <resolution>1</resolution>
-            <min_angle>-1.570796</min_angle>
-            <max_angle>1.570796</max_angle>
-          </horizontal>
-        </scan>
-        <range>
-          <min>0.10</min>
-          <max>30.0</max>
-          <resolution>0.01</resolution>
-        </range>
-        <noise>
-          <type>gaussian</type>
-          <mean>0.0</mean>
-          <stddev>0.01</stddev>
-        </noise>
-      </ray>
-      <plugin name="gazebo_ros_head_hokuyo_controller" filename="libgazebo_ros_laser.so">
-        <topicName>/ego_vehicle/laser_scan</topicName>
-        <frameName>sensor_laser</frameName>
-      </plugin>
-    </sensor>
-  </gazebo>
+    <!--Gazebo Hokuyo Laser Plugin-->
+    <gazebo reference="sensor_laser">
+        <sensor type="ray" name="head_hokuyo_sensor">
+            <pose>0 0 0 0 0 0</pose>
+            <visualize>true</visualize>
+            <update_rate>40</update_rate>
+            <ray>
+            <scan>
+                <horizontal>
+                <samples>720</samples>
+                <resolution>1</resolution>
+                <min_angle>-1.570796</min_angle>
+                <max_angle>1.570796</max_angle>
+                </horizontal>
+            </scan>
+            <range>
+                <min>0.10</min>
+                <max>30.0</max>
+                <resolution>0.01</resolution>
+            </range>
+            <noise>
+                <type>gaussian</type>
+                <mean>0.0</mean>
+                <stddev>0.01</stddev>
+            </noise>
+            </ray>
+            <plugin name="gazebo_ros_head_hokuyo_controller" filename="libgazebo_ros_laser.so">
+            <topicName>/ego_vehicle/laser_scan</topicName>
+            <frameName>sensor_laser</frameName>
+            </plugin>
+        </sensor>
+    </gazebo>
+    <!-- Gazebo Plugin for cmd_vel topic -->
+    <gazebo>
+        <plugin name="gazebo_ros_cmd_vel" filename="libgazebo_ros_planar_move.so">
+            <cmdVelTopic>/ego_vehicle/cmd_vel</cmdVelTopic>
+            <updateRate>10.0</updateRate>
+        </plugin>
+    </gazebo>
+    <!-- Gazebo Plugin for odometry topic -->
+    <gazebo>
+        <plugin name="gazebo_ros_odometry" filename="libgazebo_ros_planar_move.so">
+            <odomTopic>/ego_vehicle/odometry</odomTopic>
+            <frameId>odom</frameId>
+            <childFrameId>base_link</childFrameId>
+            <updateRate>30.0</updateRate>
+        </plugin>
+    </gazebo>
 </robot>

Commit message: getting there with the whole environment thing

File: urdf/ego_vehicle.xacro (robot description, xacro)
@@ -67,4 +67,11 @@
     </link>
     <!-- Tractor-trailer Joint -->
+    <!-- <joint name="hitch_joint" type="continuous">
+        <parent link="tractor"/>
+        <child link="trailer"/>
+        <origin xyz="0 0 0" rpy="0 0 0"/>
+        <axis xyz="0 0 1"/>
+        <limit effort="1000" velocity="1000" lower="-1.5708" upper="1.5708"/>
+    </joint> -->
     <joint name="hitch_joint" type="revolute">
         <parent link="tractor"/>
@@ -72,5 +79,5 @@
         <origin xyz="0 0 0" rpy="0 0 0"/>
         <axis xyz="0 0 1"/>
-        <limit effort="100" velocity="1.0" lower="-1.5708" upper="1.5708"/>
+        <limit effort="1000" velocity="1000.0" lower="-1.5708" upper="1.5708"/>
     </joint>
     <!-- Trailer -->

Commit message: update

File: urdf/ego_vehicle.xacro (robot description, xacro)
@@ -24,5 +24,5 @@
         </inertial>
         <visual>
-            <origin xyz="0 0 0" rpy="0 0 0" />
+            <origin xyz="0 0 0.1" rpy="0 0 0" />
             <geometry>
                 <box size="0.001 0.001 0.001" />
@@ -31,5 +31,5 @@
     </link>
     <joint name="base_footprint_joint" type="fixed">
-        <origin xyz="0 0 0" rpy="0 0 0" />
+        <origin xyz="0 0 0.1" rpy="0 0 0" />
         <parent link="base_footprint"/>
         <child link="tractor" />

File: urdf/follower_vehicle.xacro (robot description, xacro)
@@ -16,5 +16,5 @@
     <link name="base_footprint">
         <inertial>
-            <mass value="0.0001" />
+            <mass value="0.0001"/>
             <origin xyz="0 0 0" />
             <inertia ixx="0.0001" ixy="0.0" ixz="0.0"
@@ -23,5 +23,5 @@
         </inertial>
         <visual>
-            <origin xyz="0 0 0" rpy="0 0 0" />
+            <origin xyz="0 0 0.15" rpy="0 0 0" />
             <geometry>
                 <box size="0.001 0.001 0.001" />
@@ -30,5 +30,5 @@
     </link>
     <joint name="base_footprint_joint" type="fixed">
-        <origin xyz="0 0 0" rpy="0 0 0" />
+        <origin xyz="0 0 0.15" rpy="0 0 0" />
         <parent link="base_footprint"/>
         <child link="tractor" />

Commit message: updates

File: urdf/ego_vehicle.xacro (robot description, xacro)
@@ -16,11 +16,11 @@
     </xacro:macro>
     <link name="base_footprint">
-        <inertial>
+        <!-- <inertial>
             <mass value="0.0001" />
             <origin xyz="0 0 0" />
-            <inertia ixx="0.0001" ixy="0.0" ixz="0.0"
-                iyy="0.0001" iyz="0.0"
-                izz="0.0001" />
-        </inertial>
+            <inertia ixx="0.000" ixy="0.0" ixz="0.0"
+                iyy="0.000" iyz="0.0"
+                izz="0.000" />
+        </inertial> -->
         <visual>
             <origin xyz="0 0 0.1" rpy="0 0 0" />
